Commit message: update2

File: urdf/robot.urdf (robot description, URDF)
Before this commit: robot firefighting_robot, 9 links, 8 joints
Links:
- link rear_left_wheel: geometry visual cylinder length=0.015 radius=0.045
- link rear_right_wheel: geometry visual cylinder length=0.015 radius=0.045
Joints:
- joint front_left_wheel_joint: origin xyz=-0.103 0.05 0 rpy=0 1.57 0 -> xyz=-0.1105 0.05 0 rpy=0 1.57 0
- joint front_right_wheel_joint: origin xyz=0.103 0.05 0 rpy=0 1.57 0 -> xyz=0.1105 0.05 0 rpy=0 1.57 0
- joint rear_left_wheel_joint: origin xyz=-0.1 -0.1 0 rpy=0 0 0 -> xyz=-0.1105 -0.05 0 rpy=0 1.57 0
- joint rear_right_wheel_joint: origin xyz=0.1 -0.1 0 rpy=0 0 0 -> xyz=0.1105 -0.05 0 rpy=0 1.57 0

Commit message: commit

File: urdf/robot.urdf (robot description, URDF)
Before this commit: robot firefighting_robot, 9 links, 8 joints
Joints:
- joint lidar_joint: origin xyz=0 0 0.12 rpy=0 0 0 -> xyz=0 0.05 0.02 rpy=0 0 0

Commit message: odom code

File: urdf/robot.urdf (robot description, URDF)
Before this commit: robot firefighting_robot, 9 links, 8 joints
Joints:
- joint front_left_wheel_joint: axis 0 1 0 -> 0 0 1
- joint front_right_wheel_joint: axis 0 1 0 -> 0 0 1
- joint imu_joint: origin xyz=0 0 0.08 rpy=0 0 0 -> xyz=0 0 0.1 rpy=0 0 0

Commit message: midpoint, motor movement but translation erro

File: urdf/robot.urdf (robot description, URDF)
Before this commit: robot firefighting_robot, 9 links, 8 joints
Links:
- link imu: geometry visual box size=0.05 0.05 0.01
Joints:
- joint imu_joint: origin xyz=0 0 0.1 rpy=0 0 0 -> xyz=0 0.05 0 rpy=0 0 0

Commit message: urdf changes

File: urdf/robot.urdf (robot description, URDF)
Before this commit: robot firefighting_robot, 9 links, 8 joints
Links:
- removed link firehose_motor
- removed link ir_camera
- link base_link: geometry visual box size=0.20 0.206 0.052
Joints:
- removed joint firehose_motor_joint
- removed joint ir_camera_joint
- joint front_left_wheel_joint: axis 0 0 1 -> 0 0 01; origin xyz=-0.1105 0.05 0 rpy=0 1.57 0 -> xyz=0.05 0.1105 0 rpy=-1.57 1.57 0
- joint front_right_wheel_joint: origin xyz=0.1105 0.05 0 rpy=0 1.57 0 -> xyz=0.05 -0.1105 0 rpy=1.57 1.57 0
- joint imu_joint: origin xyz=0 0.05 0 rpy=0 0 0 -> xyz=0.05 0 0.0 rpy=0 0 0
- joint lidar_joint: origin xyz=0 0.05 0.02 rpy=0 0 0 -> xyz=0.05 0 0.02 rpy=0 0 0
- joint rear_left_wheel_joint: origin xyz=-0.1105 -0.05 0 rpy=0 1.57 0 -> xyz=-0.09 0.1105 0 rpy=-1.57 1.57 0
- joint rear_right_wheel_joint: origin xyz=0.1105 -0.05 0 rpy=0 1.57 0 -> xyz=-0.09 -0.1105 0 rpy=1.57 1.57 0

Commit message: urdf good

File: urdf/robot.urdf (robot description, URDF)
Before this commit: robot firefighting_robot, 7 links, 6 joints
Joints:
- joint front_left_wheel_joint: axis 0 0 01 -> 0 0 1; origin xyz=0.05 0.1105 0 rpy=-1.57 1.57 0 -> xyz=0.05 0.1105 0 rpy=1.57 1.57 0
- joint front_right_wheel_joint: origin xyz=0.05 -0.1105 0 rpy=1.57 1.57 0 -> xyz=0.05 -0.1105 0 rpy=-1.57 1.57 0

Commit message: good

File: urdf/robot.urdf (robot description, URDF)
Before this commit: robot firefighting_robot, 7 links, 6 joints
Joints:
- joint lidar_joint: origin xyz=0.05 0 0.02 rpy=0 0 0 -> xyz=0.05 0 0.089 rpy=0 0 0

Commit message: updated wheels

File: urdf/robot.urdf (robot description, URDF)
Before this commit: robot firefighting_robot, 7 links, 6 joints
Joints:
- joint front_left_wheel_joint: origin xyz=0.05 0.1105 0 rpy=1.57 1.57 0 -> xyz=0.05 0.1105 0 rpy=-1.57 1.57 0
- joint lidar_joint: origin xyz=0.05 0 0.089 rpy=0 0 0 -> xyz=0.05 0 0.089 rpy=0 0 3.1416

Commit message: good

File: urdf/robot.urdf (robot description, URDF)
Before this commit: robot firefighting_robot, 7 links, 6 joints
Joints:
- joint lidar_joint: origin xyz=0.05 0 0.089 rpy=0 0 3.1416 -> xyz=0.05 0 0.089 rpy=0 0 3.14
- joint rear_right_wheel_joint: origin xyz=-0.09 -0.1105 0 rpy=1.57 1.57 0 -> xyz=-0.09 -0.1105 0 rpy=-1.57 1.57 0

Commit message: urdf change

File: urdf/robot.urdf (robot description, URDF)
Before this commit: robot firefighting_robot, 7 links, 6 joints
Joints:
- joint lidar_joint: origin xyz=0.05 0 0.089 rpy=0 0 3.14 -> xyz=0.05 0 0.089 rpy=0 0 0

Commit message: foxy updates

File: urdf/robot.urdf (robot description, URDF)
Before this commit: robot firefighting_robot, 7 links, 6 joints
Links:
- removed link imu
- removed link lidar
- added link imu_link; visual box size=0.05 0.05 0.01
- added link lidar_link; visual cylinder length=0.02 radius=0.03
Joints:
- joint imu_joint: child imu -> imu_link
- joint lidar_joint: child lidar -> lidar_link
